Commit message: add imu and camera sensor

File: urdf/accessory/imu.xacro (robot description, xacro)
@@ -25,14 +25,18 @@
                 <visualize>true</visualize>
                 <topic>__default_topic__</topic>
-                <plugin filename="libgazebo_ros_imu_sensor.so" name="imu_plugin">
-                <topicName>imu</topicName>
-                <bodyName>$(arg ns)/imu_link</bodyName>
-                <updateRateHZ>10.0</updateRateHZ>
-                <gaussianNoise>0.0</gaussianNoise>
-                <xyzOffset>0 0 0</xyzOffset>
-                <rpyOffset>0 0 0</rpyOffset>
-                <frameName>$(arg ns)/imu_link</frameName>
-            </plugin>
-            <pose>0 0 0 0 0 0</pose>
+                <plugin filename="libgazebo_ros_imu_sensor.so" name="gazebo_imu">
+                    <ros>
+                        <namespace>$(arg ns)</namespace>
+                        <remapping>~/out:=imu</remapping>
+                    </ros>
+                    <output_type>sensor_msgs/msg/Imu</output_type>
+                    <bodyName>$(arg ns)/imu_link</bodyName>
+                    <updateRateHZ>10.0</updateRateHZ>
+                    <gaussianNoise>0.0</gaussianNoise>
+                    <xyzOffset>0 0 0</xyzOffset>
+                    <rpyOffset>0 0 0</rpyOffset>
+                    <frameName>$(arg ns)/imu_link</frameName>
+                </plugin>
+                <pose>0 0 0 0 0 0</pose>
             </sensor>
         </gazebo>

File: urdf/accessory/usb_camera.xacro (robot description, xacro)
@@ -19,5 +19,5 @@
         </gazebo>
         <gazebo reference="$(arg ns)/camera_link">
-            <sensor type="camera" name="camera_node">
+            <sensor type="camera" name="$(arg ns)/camera">
                 <update_rate>30.0</update_rate>
                 <camera name="head">

File: urdf/mrobot/main.xacro (robot description, xacro)
@@ -10,5 +10,5 @@
     <xacro:include filename="$(find my_ros2_robot_gazebo)/urdf/mrobot/caster.xacro" />
     <xacro:include filename="$(find my_ros2_robot_gazebo)/urdf/mrobot/plate.xacro" />
-    <xacro:include filename="$(find my_ros2_robot_gazebo)/urdf/accessory/rplidar.xacro" />
+    <xacro:include filename="$(find my_ros2_robot_gazebo)/urdf/accessory/lidar.xacro" />
     <xacro:include filename="$(find my_ros2_robot_gazebo)/urdf/accessory/imu.xacro" />
     <xacro:include filename="$(find my_ros2_robot_gazebo)/urdf/accessory/usb_camera.xacro" />
@@ -47,25 +47,25 @@
     <xacro:plate num="1" parent="$(arg ns)/base_link" ns="$(arg ns)" />
     <xacro:plate num="2" parent="$(arg ns)/plate_1_link" ns="$(arg ns)" />
-    <!-- Attach the Rplidar -->
-    <joint name="$(arg ns)/rplidar_joint" type="fixed">
+    <!-- Attach the lidar -->
+    <joint name="$(arg ns)/lidar_joint" type="fixed">
         <origin xyz="0 0 0.025" rpy="0 0 0" />
         <parent link="$(arg ns)/plate_2_link" />
-        <child link="$(arg ns)/rplidar_link" />
+        <child link="$(arg ns)/lidar_link" />
     </joint>
-    <xacro:rplidar ns="$(arg ns)" />
+    <xacro:lidar ns="$(arg ns)" />
     <!-- Attach the IMU -->
-    <!-- <joint name="$(arg ns)/imu_joint" type="fixed">
+    <joint name="$(arg ns)/imu_joint" type="fixed">
         <origin xyz="0 0 0.02" rpy="0 0 0" />
         <parent link="$(arg ns)/base_link" />
         <child link="$(arg ns)/imu_link" />
     </joint>
-    <xacro:imu ns="$(arg ns)" /> -->
+    <xacro:imu ns="$(arg ns)" />
     <!-- Attach the Camera -->
-    <!-- <joint name="$(arg ns)/camera_joint" type="fixed">
+    <joint name="$(arg ns)/camera_joint" type="fixed">
         <origin xyz="0.12 0 0.1" rpy="0 0 0" />
         <parent link="$(arg ns)/base_link" />
         <child link="$(arg ns)/camera_link" />
     </joint>
-    <xacro:usb_camera ns="$(arg ns)" /> -->
+    <xacro:usb_camera ns="$(arg ns)" />
     <!-- # joint state -->
     <gazebo>
