Commit message: add slam

File: urdf/accessory/lidar.xacro (robot description, xacro)
@@ -21,5 +21,5 @@
             <sensor name="$(arg ns)/lidar_sensor" type="ray">
                 <always_on>true</always_on>
-                <visualize>true</visualize>
+                <visualize>false</visualize>
                 <pose>0.0 0 0 0 0 0</pose>
                 <update_rate>5</update_rate>

File: urdf/mrobot/main.xacro (robot description, xacro)
@@ -44,4 +44,5 @@
     <!-- Casters Definitions -->
     <xacro:caster fb="front"  translateX="1" parent="$(arg ns)/base_link" ns="$(arg ns)" />
+    <xacro:caster fb="back"  translateX="-1" parent="$(arg ns)/base_link" ns="$(arg ns)" />
     <!-- plate Definitions -->
     <xacro:plate num="1" parent="$(arg ns)/base_link" ns="$(arg ns)" />
@@ -107,5 +108,5 @@
             <robot_base_frame>base_link</robot_base_frame>
             <!-- Odometry source, 0 for ENCODER, 1 for WORLD, defaults to WORLD -->
-            <odometry_source>0</odometry_source>
+            <odometry_source>1</odometry_source>
             <!-- Change the ROS topic we will publish the odometry data to -->
             <ros>

File: urdf/mrobot/property.xacro (robot description, xacro)
@@ -7,5 +7,5 @@
     <xacro:property name="base_link_radius" value="0.13"/>
     <xacro:property name="base_link_length" value="0.005"/>
-    <xacro:property name="motor_x" value="-0.05"/>
+    <xacro:property name="motor_x" value="0.0"/>
     <!-- Wheel radius, height and mass -->
     <xacro:property name="wheel_radius" value="0.033" />

File: urdf/mrobot/wheel.xacro (robot description, xacro)
@@ -7,5 +7,5 @@
             <parent link="${parent}"/>
             <child link="$(arg ns)/wheel_${lr}_link"/>
-            <origin xyz="${motor_x} ${translateY * base_link_radius} 0" rpy="0 0 0" />
+            <origin xyz="${motor_x} ${translateY * (base_link_radius + wheel_height/2)} 0" rpy="0 0 0" />
             <axis xyz="0 1 0" rpy="0 0 0" />
         </joint>
