Commit message: add namespace

File: urdf/accessory/camera_m.xacro (robot description, xacro)
@@ -19,26 +19,30 @@
         </gazebo>
         <gazebo reference="$(arg ns)/camera_link">
-            <sensor name='$(arg ns)/camera_sensor' type='camera'>
+            <sensor name='camera_topics' type='camera'>
+                <plugin name='camera_driver' filename='libgazebo_ros_camera.so'>
+                    <ros>
+                        <namespace>$(arg ns)</namespace>
+                    </ros>
+                </plugin>
                 <always_on>1</always_on>
                 <visualize>0</visualize>
                 <update_rate>30</update_rate>
                 <camera name='$(arg ns)/camera'>
-                <horizontal_fov>1.0856</horizontal_fov>
-                <image>
-                    <width>1280</width>
-                    <height>720</height>
-                    <format>R8G8B8</format>
-                </image>
-                <clip>
-                    <near>0.03</near>
-                    <far>100</far>
-                </clip>
-                <noise>
-                    <type>gaussian</type>
-                    <mean>0</mean>
-                    <stddev>0.007</stddev>
-                </noise>
+                    <horizontal_fov>1.0856</horizontal_fov>
+                    <image>
+                        <width>1280</width>
+                        <height>720</height>
+                        <format>R8G8B8</format>
+                    </image>
+                    <clip>
+                        <near>0.03</near>
+                        <far>100</far>
+                    </clip>
+                    <noise>
+                        <type>gaussian</type>
+                        <mean>0</mean>
+                        <stddev>0.007</stddev>
+                    </noise>
                 </camera>
-                <plugin name='camera_driver' filename='libgazebo_ros_camera.so'/>
             </sensor>
         </gazebo>

File: urdf/accessory/lidar.xacro (robot description, xacro)
@@ -19,5 +19,5 @@
         </gazebo>
         <gazebo reference="$(arg ns)/lidar_link">
-            <sensor name="$(arg ns)/lidar_sensor" type="ray">
+            <sensor name="$(arg ns)/lidar_link" type="ray">
                 <always_on>true</always_on>
                 <visualize>false</visualize>
@@ -45,10 +45,16 @@
                 </ray>
                 <plugin name="gazebo_lidar" filename="libgazebo_ros_ray_sensor.so">
+                    <output_type>sensor_msgs/LaserScan</output_type>
+                    <!-- use /lidar_link for frame_name will have error -->
+                    <xacro:if value="${ns == ''}">
+                        <frame_name>lidar_link</frame_name>
+                    </xacro:if>
+                    <xacro:unless value="${ns == ''}">
+                        <frame_name>$(arg ns)/lidar_link</frame_name>
+                    </xacro:unless>
                     <ros>
                         <namespace>$(arg ns)</namespace>
                         <remapping>~/out:=scan</remapping>
                     </ros>
-                    <output_type>sensor_msgs/LaserScan</output_type>
-                    <frame_name>lidar_link</frame_name>
                 </plugin>
             </sensor>

File: urdf/mrobot/main.xacro (robot description, xacro)
@@ -21,5 +21,5 @@
     <xacro:include filename="../accessory/lidar.xacro" />
     <xacro:include filename="../accessory/imu.xacro" />
-    <xacro:include filename="../accessory/camera_m.xacro" />
+    <!-- <xacro:include filename="../accessory/camera_m.xacro" /> -->
     <!-- Body of robot, with plates, standoffs and Create -->
     <!-- BASE-LINK -->
@@ -72,15 +72,16 @@
     <xacro:imu ns="$(arg ns)" />
     <!-- Attach the Camera -->
-    <joint name="$(arg ns)/camera_joint" type="fixed">
+    <!-- <joint name="$(arg ns)/camera_joint" type="fixed">
         <origin xyz="0.12 0 0.1" rpy="0 0 0" />
         <parent link="$(arg ns)/base_link" />
         <child link="$(arg ns)/camera_link" />
     </joint>
-    <xacro:camera_m ns="$(arg ns)" />
+    <xacro:camera_m ns="$(arg ns)" /> -->
     <!-- # joint state -->
     <gazebo>
         <plugin name="joint_state_publisher" filename="libgazebo_ros_joint_state_publisher.so">
             <ros>
-                <remapping>~/out:=joint_states</remapping>
+                <namespace>$(arg ns)</namespace>
+                <remapping>~/out:=$(arg ns)/joint_states</remapping>
             </ros>
             <update_rate>30</update_rate>
@@ -93,6 +94,7 @@
         <plugin name='differential_drive_controller' filename='libgazebo_ros_diff_drive.so'>
             <ros>
-              <!-- <remapping>cmd_vel:=cmd_vel</remapping> -->
-              <!-- <remapping>odom:=odom</remapping> -->
+                <namespace>$(arg ns)</namespace>
+                <!-- <remapping>cmd_vel:=cmd_vel</remapping> -->
+                <!-- <remapping>odom:=odom</remapping> -->
             </ros>
             <!-- wheels -->
@@ -109,6 +111,6 @@
             <publish_odom_tf>true</publish_odom_tf>
             <publish_wheel_tf>true</publish_wheel_tf>
-            <odometry_frame>odom</odometry_frame>
-            <robot_base_frame>base_link</robot_base_frame>
+            <odometry_frame>$(arg ns)/odom</odometry_frame>
+            <robot_base_frame>$(arg ns)/base_link</robot_base_frame>
         </plugin>
     </gazebo>
